Commit message: Add xacro expansion into CMakeLists.txt.

File: urdf/model.urdf (robot description, URDF)
Before this commit: robot rrbot, 5 links, 4 joints
Links:
- link base_link: mass 0.01 -> 10
- link link1: mass 0.01 -> 10
- link link2: mass 0.01 -> 10

File: urdf/model.urdf.xacro (robot description, xacro)
@@ -5,7 +5,10 @@
 <robot xmlns:xacro="http://wiki.ros.org/xacro" name="rrbot">
   <!-- ======================================== -->
-  <!-- launchファイル経由で設定するパラメータ引数   -->
+  <!-- CMakeによるurdf生成用                     -->
   <!-- ======================================== -->
-  <!-- ハードウェア利用フラグ -->
+  <xacro:arg name="project_dir" default="$(find rrbot_description)" />
+  <!-- ======================================== -->
+  <!-- ハードウェア利用フラグ                     -->
+  <!-- ======================================== -->
   <xacro:arg name="use_mock" default="false" />
   <xacro:arg name="use_gazebo" default="false" />
@@ -20,10 +23,12 @@
   <!-- ======================================== -->
   <!-- ロボットの定義 -->
-  <xacro:include filename="$(find rrbot_description)/urdf/rrbot.xacro" />
+  <xacro:include filename="$(arg project_dir)/urdf/rrbot.xacro" />
+  <xacro:include filename="$(arg project_dir)/urdf/inertial.xacro" />
+  <xacro:include filename="$(arg project_dir)/urdf/material.xacro" />
   <xacro:rrbot parent="world">
     <origin xyz="0.0 0.0 0.0" rpy="0.0 0.0 0.0" />
   </xacro:rrbot>
   <!-- ros2_controlの定義 -->
-  <xacro:include filename="$(find rrbot_description)/urdf/rrbot_control.xacro" />
+  <xacro:include filename="$(arg project_dir)/urdf/rrbot_control.xacro" />
   <xacro:rrbot_control
     use_mock="$(arg use_mock)"

File: urdf/rrbot.xacro (robot description, xacro)
@@ -4,6 +4,4 @@
 <!-- ======================================== -->
 <robot xmlns:xacro="http://wiki.ros.org/xacro">
-  <xacro:include filename="$(find rrbot_description)/urdf/inertial.xacro" />
-  <xacro:include filename="$(find rrbot_description)/urdf/material.xacro" />
   <!-- args
     parent: ロボットの親座標系の名前
