Commit message: Fix inertia origin problem in xacro files.

File: urdf/inertial.xacro (robot description, xacro)
@@ -5,9 +5,7 @@
 <robot xmlns:xacro="http://wiki.ros.org/xacro">
   <!-- 慣性のデフォルト値 -->
-  <xacro:macro name="default_inertial">
+  <xacro:macro name="default_inertial" params="*origin">
     <inertial>
-      <origin
-        xyz="0.0 0.0 0.0"
-        rpy="0.0 0.0 0.0" />
+      <xacro:insert_block name="origin" />
       <mass
         value="0.01" />

File: urdf/rrbot.xacro (robot description, xacro)
@@ -17,6 +17,8 @@
     <link name="base_link">
       <!-- 形状定義 -->
+      <xacro:property name="base_link_origin">
+        <origin xyz="0.0 0.0 0.15" rpy="0.0 0.0 0.0" />
+      </xacro:property>
       <xacro:property name="base_link_shape">
-        <origin xyz="0.0 0.0 0.15" rpy="0.0 0.0 0.0" />
         <geometry>
           <box size="0.3 0.3 0.3" />
@@ -24,17 +26,23 @@
       </xacro:property>
       <visual>
+        <xacro:insert_block name="base_link_origin" />
         <xacro:insert_block name="base_link_shape" />
         <material name="red" />
       </visual>
       <collision>
+        <xacro:insert_block name="base_link_origin" />
         <xacro:insert_block name="base_link_shape" />
       </collision>
-      <xacro:default_inertial />
+      <xacro:default_inertial>
+        <xacro:insert_block name="base_link_origin" />
+      </xacro:default_inertial>
     </link>
     <!-- link1 -->
     <link name="link1">
       <!-- 形状定義 -->
+      <xacro:property name="link1_origin">
+        <origin xyz="0.0 0.0 0.25" rpy="0.0 0.0 0.0" />
+      </xacro:property>
       <xacro:property name="link1_shape">
-        <origin xyz="0.0 0.0 0.25" rpy="0.0 0.0 0.0" />
         <geometry>
           <cylinder length="0.5" radius="${0.2 / 2.0}" />
@@ -42,17 +50,23 @@
       </xacro:property>
       <visual>
+        <xacro:insert_block name="link1_origin" />
         <xacro:insert_block name="link1_shape" />
         <material name="green" />
       </visual>
       <collision>
+        <xacro:insert_block name="link1_origin" />
         <xacro:insert_block name="link1_shape" />
       </collision>
-      <xacro:default_inertial />
+      <xacro:default_inertial>
+        <xacro:insert_block name="link1_origin" />
+      </xacro:default_inertial>
     </link>
     <!-- link 2 -->
     <link name="link2">
       <!-- 形状定義 -->
+      <xacro:property name="link2_origin">
+        <origin xyz="0.0 0.0 0.3" rpy="0.0 0.0 0.0" />
+      </xacro:property>
       <xacro:property name="link2_shape">
-        <origin xyz="0.0 0.0 0.3" rpy="0.0 0.0 0.0" />
         <geometry>
           <box size="0.1 0.1 0.6" />
@@ -60,11 +74,15 @@
       </xacro:property>
       <visual>
+        <xacro:insert_block name="link2_origin" />
         <xacro:insert_block name="link2_shape" />
         <material name="blue" />
       </visual>
       <collision>
+        <xacro:insert_block name="link2_origin" />
         <xacro:insert_block name="link2_shape" />
       </collision>
-      <xacro:default_inertial />
+      <xacro:default_inertial>
+        <xacro:insert_block name="link2_origin" />
+      </xacro:default_inertial>
     </link>
     <!-- tool0 -->

Commit message: Change structure of xacro files.

File: urdf/inertial.xacro (robot description, xacro)
@@ -1,21 +1,17 @@
 <?xml version="1.0" encoding="UTF-8"?>
-<!-- ======================================== -->
-<!-- 慣性定義                                   -->
-<!-- ======================================== -->
 <robot xmlns:xacro="http://wiki.ros.org/xacro">
-  <!-- 慣性のデフォルト値 -->
-  <xacro:macro name="default_inertial" params="*origin">
-    <inertial>
-      <xacro:insert_block name="origin" />
-      <mass
-        value="10" />
-      <inertia
-        ixx="0.05"
-        iyy="0.05"
-        izz="0.05"
-        ixy="0.0"
-        iyz="0.0"
-        ixz="0.0" />
-    </inertial>
+  <!-- ======================================== -->
+  <!-- 慣性のデフォルト値                         -->
+  <!-- ======================================== -->
+  <xacro:macro name="default_inertial">
+    <mass
+      value="10" />
+    <inertia
+      ixx="0.05"
+      iyy="0.05"
+      izz="0.05"
+      ixy="0.0"
+      iyz="0.0"
+      ixz="0.0" />
   </xacro:macro>
 </robot>

File: urdf/material.xacro (robot description, xacro)
@@ -1,7 +1,7 @@
 <?xml version="1.0" encoding="UTF-8"?>
-<!-- ======================================== -->
-<!-- 材質定義                                   -->
-<!-- ======================================== -->
 <robot xmlns:xacro="http://wiki.ros.org/xacro">
+  <!-- ======================================== -->
+  <!-- 材質定義                                   -->
+  <!-- ======================================== -->
   <material name="red">
     <color rgba="1.0 0.0 0.0 1.0" />

File: urdf/model.urdf.xacro (robot description, xacro)
@@ -1,11 +1,4 @@
 <?xml version="1.0" encoding="UTF-8"?>
-<!-- ======================================== -->
-<!-- URDF本体                                 -->
-<!-- ======================================== -->
 <robot xmlns:xacro="http://wiki.ros.org/xacro" name="rrbot">
-  <!-- ======================================== -->
-  <!-- CMakeによるurdf生成用                     -->
-  <!-- ======================================== -->
-  <xacro:arg name="project_dir" default="$(find rrbot_description)" />
   <!-- ======================================== -->
   <!-- ハードウェア利用フラグ                     -->
@@ -20,15 +13,20 @@
   <link name="world" />
   <!-- ======================================== -->
-  <!-- rrbotの定義                             -->
+  <!-- ロボットの形状定義                         -->
   <!-- ======================================== -->
-  <!-- ロボットの定義 -->
-  <xacro:include filename="$(arg project_dir)/urdf/rrbot.xacro" />
-  <xacro:include filename="$(arg project_dir)/urdf/inertial.xacro" />
-  <xacro:include filename="$(arg project_dir)/urdf/material.xacro" />
-  <xacro:rrbot parent="world">
+  <!--  parent:         ロボットの親座標系の名前
+        parent_origin:  ロボットの親座標系の原点  -->
+  <xacro:include filename="rrbot.xacro" />
+  <xacro:rrbot
+    parent="world">
     <origin xyz="0.0 0.0 0.0" rpy="0.0 0.0 0.0" />
   </xacro:rrbot>
-  <!-- ros2_controlの定義 -->
-  <xacro:include filename="$(arg project_dir)/urdf/rrbot_control.xacro" />
+  <!-- ======================================== -->
+  <!-- ros2_control定義                         -->
+  <!-- ======================================== -->
+  <!--  use_mock:     モックハードウェア利用フラグ
+        use_gazebo:   Gazebo利用フラグ
+        use_unity:    Unity利用フラグ   -->
+  <xacro:include filename="rrbot_control.xacro" />
   <xacro:rrbot_control
     use_mock="$(arg use_mock)"

File: urdf/rrbot.xacro (robot description, xacro)
@@ -1,12 +1,7 @@
 <?xml version="1.0" encoding="UTF-8"?>
-<!-- ======================================== -->
-<!-- ロボットの形状定義                         -->
-<!-- ======================================== -->
 <robot xmlns:xacro="http://wiki.ros.org/xacro">
-  <!-- args
-    parent: ロボットの親座標系の名前
-    origin: ロボットの親座標系の原点
-  -->
-  <xacro:macro name="rrbot" params="parent *origin">
+  <xacro:macro name="rrbot" params="parent *parent_origin">
+    <xacro:include filename="inertial.xacro" />
+    <xacro:include filename="material.xacro" />
     <!-- ======================================== -->
     <!-- Linkages                                 -->
@@ -14,73 +9,91 @@
     <!-- base_link -->
     <link name="base_link">
-      <!-- 形状定義 -->
-      <xacro:property name="base_link_origin">
+      <!-- 原点 -->
+      <xacro:property name="origin">
         <origin xyz="0.0 0.0 0.15" rpy="0.0 0.0 0.0" />
       </xacro:property>
-      <xacro:property name="base_link_shape">
+      <!-- 形状 -->
+      <xacro:property name="shape">
         <geometry>
           <box size="0.3 0.3 0.3" />
         </geometry>
       </xacro:property>
+      <!-- 慣性 -->
+      <xacro:property name="inertial">
+        <xacro:default_inertial />
+      </xacro:property>
       <visual>
-        <xacro:insert_block name="base_link_origin" />
-        <xacro:insert_block name="base_link_shape" />
+        <xacro:insert_block name="origin" />
+        <xacro:insert_block name="shape" />
         <material name="red" />
       </visual>
       <collision>
-        <xacro:insert_block name="base_link_origin" />
-        <xacro:insert_block name="base_link_shape" />
+        <xacro:insert_block name="origin" />
+        <xacro:insert_block name="shape" />
       </collision>
-      <xacro:default_inertial>
-        <xacro:insert_block name="base_link_origin" />
-      </xacro:default_inertial>
+      <inertial>
+        <xacro:insert_block name="origin" />
+        <xacro:insert_block name="inertial" />
+      </inertial>
     </link>
     <!-- link1 -->
     <link name="link1">
-      <!-- 形状定義 -->
-      <xacro:property name="link1_origin">
+      <!-- 原点 -->
+      <xacro:property name="origin">
         <origin xyz="0.0 0.0 0.25" rpy="0.0 0.0 0.0" />
       </xacro:property>
-      <xacro:property name="link1_shape">
+      <!-- 形状 -->
+      <xacro:property name="shape">
         <geometry>
           <cylinder length="0.5" radius="${0.2 / 2.0}" />
         </geometry>
       </xacro:property>
+      <!-- 慣性 -->
+      <xacro:property name="inertial">
+        <xacro:default_inertial />
+      </xacro:property>
       <visual>
-        <xacro:insert_block name="link1_origin" />
-        <xacro:insert_block name="link1_shape" />
+        <xacro:insert_block name="origin" />
+        <xacro:insert_block name="shape" />
         <material name="green" />
       </visual>
       <collision>
-        <xacro:insert_block name="link1_origin" />
-        <xacro:insert_block name="link1_shape" />
+        <xacro:insert_block name="origin" />
+        <xacro:insert_block name="shape" />
       </collision>
-      <xacro:default_inertial>
-        <xacro:insert_block name="link1_origin" />
-      </xacro:default_inertial>
+      <inertial>
+        <xacro:insert_block name="origin" />
+        <xacro:insert_block name="inertial" />
+      </inertial>
     </link>
     <!-- link 2 -->
     <link name="link2">
-      <!-- 形状定義 -->
-      <xacro:property name="link2_origin">
+      <!-- 原点 -->
+      <xacro:property name="origin">
         <origin xyz="0.0 0.0 0.3" rpy="0.0 0.0 0.0" />
       </xacro:property>
-      <xacro:property name="link2_shape">
+      <!-- 形状 -->
+      <xacro:property name="shape">
         <geometry>
           <box size="0.1 0.1 0.6" />
         </geometry>
       </xacro:property>
+      <!-- 慣性 -->
+      <xacro:property name="inertial">
+        <xacro:default_inertial />
+      </xacro:property>
       <visual>
-        <xacro:insert_block name="link2_origin" />
-        <xacro:insert_block name="link2_shape" />
+        <xacro:insert_block name="origin" />
+        <xacro:insert_block name="shape" />
         <material name="blue" />
       </visual>
       <collision>
-        <xacro:insert_block name="link2_origin" />
-        <xacro:insert_block name="link2_shape" />
+        <xacro:insert_block name="origin" />
+        <xacro:insert_block name="shape" />
       </collision>
-      <xacro:default_inertial>
-        <xacro:insert_block name="link2_origin" />
-      </xacro:default_inertial>
+      <inertial>
+        <xacro:insert_block name="origin" />
+        <xacro:insert_block name="inertial" />
+      </inertial>
     </link>
     <!-- tool0 -->
@@ -93,5 +106,5 @@
       <parent link="${parent}" />
       <child link="base_link" />
-      <xacro:insert_block name="origin" />
+      <xacro:insert_block name="parent_origin" />
     </joint>
     <!-- joint1 (base_link -> link1) -->

File: urdf/rrbot_control.xacro (robot description, xacro)
@@ -1,14 +1,9 @@
 <?xml version="1.0" encoding="UTF-8"?>
-<!-- ======================================== -->
-<!-- ros2_control用                           -->
-<!-- ======================================== -->
 <robot xmlns:xacro="http://wiki.ros.org/xacro">
-  <!-- args
-    use_mock: モックハードウェア利用フラグ
-    use_gazebo: Gazebo利用フラグ
-    use_unity: Unity利用フラグ
-  -->
   <xacro:macro name="rrbot_control"
     params="use_mock:=^|false use_gazebo:=^|false use_unity:=^|false">
+    <!-- ======================================== -->
+    <!-- ros2_control                             -->
+    <!-- ======================================== -->
     <ros2_control name="rrbot" type="system">
       <!-- ======================================== -->

Commit message: Linkage definitions are made macro.

File: urdf/inertial.xacro (robot description, xacro)
@@ -5,5 +5,5 @@
   <!-- ======================================== -->
   <!-- Simple inertial value for testing -->
-  <xacro:macro name="default_inertial">
+  <xacro:property name="default_inertial">
     <mass
       value="10" />
@@ -15,4 +15,4 @@
       iyz="0.0"
       ixz="0.0" />
-  </xacro:macro>
+  </xacro:property>
 </robot>

File: urdf/rrbot.xacro (robot description, xacro)
@@ -8,7 +8,12 @@
     parent_origin:  origin of parent coordination
   -->
-  <xacro:macro name="rrbot" params="parent *parent_origin">
+  <xacro:macro name="rrbot"
+    params="parent *parent_origin">
+    <!-- ======================================== -->
+    <!-- Include macros                           -->
+    <!-- ======================================== -->
     <xacro:include filename="material.xacro" />
     <xacro:include filename="inertial.xacro" />
+    <xacro:include filename="linkage.xacro" />
     <!-- ======================================== -->
     <!-- Linkages                                 -->
@@ -16,91 +21,34 @@
     <!-- base_link -->
     <link name="base_link">
-      <!-- origin -->
-      <xacro:property name="origin">
+      <xacro:linkage>
         <origin xyz="0.0 0.0 0.15" rpy="0.0 0.0 0.0" />
-      </xacro:property>
-      <!-- shape -->
-      <xacro:property name="shape">
         <geometry>
           <box size="0.3 0.3 0.3" />
         </geometry>
-      </xacro:property>
-      <!-- inertial -->
-      <xacro:property name="inertial">
-        <xacro:default_inertial />
-      </xacro:property>
-      <visual>
-        <xacro:insert_block name="origin" />
-        <xacro:insert_block name="shape" />
+        <xacro:insert_block name="default_inertial" />
         <material name="red" />
-      </visual>
-      <collision>
-        <xacro:insert_block name="origin" />
-        <xacro:insert_block name="shape" />
-      </collision>
-      <inertial>
-        <xacro:insert_block name="origin" />
-        <xacro:insert_block name="inertial" />
-      </inertial>
+      </xacro:linkage>
     </link>
     <!-- link1 -->
     <link name="link1">
-      <!-- origin -->
-      <xacro:property name="origin">
+      <xacro:linkage>
         <origin xyz="0.0 0.0 0.25" rpy="0.0 0.0 0.0" />
-      </xacro:property>
-      <!-- shape -->
-      <xacro:property name="shape">
         <geometry>
           <cylinder length="0.5" radius="${0.2 / 2.0}" />
         </geometry>
-      </xacro:property>
-      <!-- inertial -->
-      <xacro:property name="inertial">
-        <xacro:default_inertial />
-      </xacro:property>
-      <visual>
-        <xacro:insert_block name="origin" />
-        <xacro:insert_block name="shape" />
+        <xacro:insert_block name="default_inertial" />
         <material name="green" />
-      </visual>
-      <collision>
-        <xacro:insert_block name="origin" />
-        <xacro:insert_block name="shape" />
-      </collision>
-      <inertial>
-        <xacro:insert_block name="origin" />
-        <xacro:insert_block name="inertial" />
-      </inertial>
+      </xacro:linkage>
     </link>
     <!-- link 2 -->
     <link name="link2">
-      <!-- origin -->
-      <xacro:property name="origin">
+      <xacro:linkage>
         <origin xyz="0.0 0.0 0.3" rpy="0.0 0.0 0.0" />
-      </xacro:property>
-      <!-- shape -->
-      <xacro:property name="shape">
         <geometry>
           <box size="0.1 0.1 0.6" />
         </geometry>
-      </xacro:property>
-      <!-- inertial -->
-      <xacro:property name="inertial">
-        <xacro:default_inertial />
-      </xacro:property>
-      <visual>
-        <xacro:insert_block name="origin" />
-        <xacro:insert_block name="shape" />
+        <xacro:insert_block name="default_inertial" />
         <material name="blue" />
-      </visual>
-      <collision>
-        <xacro:insert_block name="origin" />
-        <xacro:insert_block name="shape" />
-      </collision>
-      <inertial>
-        <xacro:insert_block name="origin" />
-        <xacro:insert_block name="inertial" />
-      </inertial>
+      </xacro:linkage>
     </link>
     <!-- tool0 -->

Commit message: Change robot inertial parameters.

File: urdf/inertial.xacro (robot description, xacro)
@@ -7,9 +7,9 @@
   <xacro:property name="default_inertial">
     <mass
-      value="10" />
+      value="1" />
     <inertia
-      ixx="0.05"
-      iyy="0.05"
-      izz="0.05"
+      ixx="0.01"
+      iyy="0.01"
+      izz="0.01"
       ixy="0.0"
       iyz="0.0"

File: urdf/model.urdf (robot description, URDF)
Before this commit: robot rrbot, 5 links, 4 joints
Links:
- link base_link: mass 10 -> 1
- link link1: mass 10 -> 1
- link link2: mass 10 -> 1
Joints:
- joint joint1: limit lower=-6.632251157578453 upper=6.632251157578453 effort=1.0 velocity=3.141592653589793 -> lower=-6.632251157578453 upper=6.632251157578453 effort=10.0 velocity=3.141592653589793
- joint joint2: limit lower=-1.0471975511965976 upper=4.1887902047863905 effort=1.0 velocity=3.141592653589793 -> lower=-1.0471975511965976 upper=4.1887902047863905 effort=10.0 velocity=3.141592653589793

File: urdf/rrbot.xacro (robot description, xacro)
@@ -70,9 +70,9 @@
       <axis xyz="0.0 0.0 1.0" />
       <limit
-        effort="1.0"
+        effort="10.0"
         lower="${radians(-380.0)}"
         upper="${radians(380.0)}"
         velocity="${radians(180.0)}" />
-      <dynamics damping="0.01" friction="0.0" />
+      <dynamics damping="0.1" friction="0.0" />
     </joint>
     <!-- joint2 (link1 -> link2) -->
@@ -83,9 +83,9 @@
       <axis xyz="0.0 1.0 0.0" />
       <limit
-        effort="1.0"
+        effort="10.0"
         lower="${radians(-60.0)}"
         upper="${radians(240.0)}"
         velocity="${radians(180.0)}" />
-      <dynamics damping="0.01" friction="0.0" />
+      <dynamics damping="0.1" friction="0.0" />
     </joint>
     <!-- joint3 (link2 -> tool0) -->
